Commit message: Creation of urdf

File: etarobtest/urdf/base.urdf.xacro (robot description, xacro)
@@ -106,5 +106,5 @@
   <xacro:macro name= "base_lower" params="suffix *origin rot_axis">
     <joint name= "${suffix}_base_lower" type="revolute">
-       <axis xyz="0 ${rot_axis} 0" />-->
+       <axis xyz="0 ${rot_axis} 0" />
        <limit lower="${-5*M_PI/180.0}" upper="${5*M_PI/180.0}" effort="${10*mx160_effort}" velocity="${mx160_velocity/5}"/>
        <parent link="base_link" />

Commit message: Add files via upload

File: etarobtest/urdf/base.urdf.xacro (robot description, xacro)
@@ -163,5 +163,5 @@
     </link>
   </xacro:macro>
-  <!--arm_connection_lower -->
+  <!--arm_connection_lower
   <xacro:macro name= "arm_connection_lower" params="suffix rot_axis">
     <joint name= "${suffix}_lower_joint" type="revolute">
@@ -170,5 +170,5 @@
        <child link="${suffix}_arm" />
     </joint>
-  </xacro:macro>
+  </xacro:macro> -->
   <!-- wheel -->
   <xacro:macro name="odom_wheel_tire" params="*origin suffix rot_axis_wheel">
@@ -237,8 +237,8 @@
     <origin xyz="1.194088 0.214831 -1.006421" rpy="0 0 0" />
   </xacro:arm_connection_upper>
-  <xacro:arm_connection_lower suffix="fl" rot_axis="1" />
+  <!--<xacro:arm_connection_lower suffix="fl" rot_axis="1" />
   <xacro:arm_connection_lower suffix="fr" rot_axis="-1" />
   <xacro:arm_connection_lower suffix="bl" rot_axis="1" />
-  <xacro:arm_connection_lower suffix="br" rot_axis="1" />
+  <xacro:arm_connection_lower suffix="br" rot_axis="1" />-->
   <!--<xacro:arm_connection_upper suffix="fl" rot_axis="1" >
     <origin xyz="0 0 0" rpy="0 0 0" />

Commit message: Addition of Transmission elements

File: etarobtest/urdf/base.urdf.xacro (robot description, xacro)
@@ -200,4 +200,5 @@
       </collision>
     </link>
+    <xacro:gazebo_wheel_link name="${suffix}_wheel_link"/>
   </xacro:macro>
   <xacro:base_upper suffix="fl" rot_axis="1" >

File: etarobtest/urdf/test.gazebo.xacro (robot description, xacro)
@@ -24,5 +24,5 @@
     <material>Gazebo/Grey</material>
   </gazebo>
-  <xacro:macro name="odom_wheel_tire" params="name">
+  <xacro:macro name="gazebo_wheel_link" params="name">
     <gazebo reference="${name}">
       <kp>100000.0</kp>

Commit message: Addition of Transmission elements

File: etarobtest/urdf/base.urdf.xacro (robot description, xacro)
@@ -163,5 +163,5 @@
     </link>
   </xacro:macro>
-  <!--arm_connection_lower
+  <!--arm_connection_lower-->
   <xacro:macro name= "arm_connection_lower" params="suffix rot_axis">
     <joint name= "${suffix}_lower_joint" type="revolute">
@@ -170,5 +170,5 @@
        <child link="${suffix}_arm" />
     </joint>
-  </xacro:macro> -->
+  </xacro:macro>
   <!-- wheel -->
   <xacro:macro name="odom_wheel_tire" params="*origin suffix rot_axis_wheel">
@@ -238,8 +238,8 @@
     <origin xyz="1.194088 0.214831 -1.006421" rpy="0 0 0" />
   </xacro:arm_connection_upper>
-  <!--<xacro:arm_connection_lower suffix="fl" rot_axis="1" />
+  <xacro:arm_connection_lower suffix="fl" rot_axis="1" />
   <xacro:arm_connection_lower suffix="fr" rot_axis="-1" />
   <xacro:arm_connection_lower suffix="bl" rot_axis="1" />
-  <xacro:arm_connection_lower suffix="br" rot_axis="1" />-->
+  <xacro:arm_connection_lower suffix="br" rot_axis="1" />
   <!--<xacro:arm_connection_upper suffix="fl" rot_axis="1" >
     <origin xyz="0 0 0" rpy="0 0 0" />

Commit message: Addition of transmission element

File: etarobtest/urdf/base.urdf.xacro (robot description, xacro)
@@ -164,9 +164,11 @@
   </xacro:macro>
   <!--arm_connection_lower-->
-  <xacro:macro name= "arm_connection_lower" params="suffix rot_axis">
+  <xacro:macro name= "arm_connection_lower" params="suffix *origin rot_axis">
     <joint name= "${suffix}_lower_joint" type="revolute">
+       <axis xyz="0 ${rot_axis} 0" />
        <limit lower="${-5*M_PI/180.0}" upper="${5*M_PI/180.0}" effort="${10*mx160_effort}" velocity="${mx160_velocity/5}"/>
        <parent link="${suffix}_connection_lower" />
        <child link="${suffix}_arm" />
+       <xacro:insert_block name="origin" />
     </joint>
     <xacro:simple_transmission name="${suffix}_lower_joint" interface="hardware_interface/EffortJointInterface" />
@@ -239,8 +241,20 @@
     <origin xyz="1.194088 0.214831 -1.006421" rpy="0 0 0" />
   </xacro:arm_connection_upper>
-  <xacro:arm_connection_lower suffix="fl" rot_axis="1" />
+    <!--<xacro:arm_connection_lower suffix="fl" rot_axis="1" />
   <xacro:arm_connection_lower suffix="fr" rot_axis="-1" />
   <xacro:arm_connection_lower suffix="bl" rot_axis="1" />
-  <xacro:arm_connection_lower suffix="br" rot_axis="1" />
+  <xacro:arm_connection_lower suffix="br" rot_axis="1" />-->
+  <xacro:arm_connection_lower suffix="fl" rot_axis="1" >
+    <origin xyz="0 0 0" rpy="0 0 0" />
+  </xacro:arm_connection_lower>
+  <xacro:arm_connection_lower suffix="fr" rot_axis="-1" >
+    <origin xyz="0 0 0" rpy="0 0 0" />
+  </xacro:arm_connection_lower>
+  <xacro:arm_connection_lower suffix="bl" rot_axis="1" >
+    <origin xyz="0 0 0" rpy="0 0 0" />
+  </xacro:arm_connection_lower>
+  <xacro:arm_connection_lower suffix="br" rot_axis="1" >
+    <origin xyz="0 0 0" rpy="0 0 0" />
+  </xacro:arm_connection_lower>
   <!--<xacro:arm_connection_upper suffix="fl" rot_axis="1" >
     <origin xyz="0 0 0" rpy="0 0 0" />

File: etarobtest/urdf/test.gazebo.xacro (robot description, xacro)
@@ -73,6 +73,6 @@
       </joint>
       <actuator name="${name}_motor">
+        <hardwareInterface>${interface}</hardwareInterface>
         <mechanicalReduction>10</mechanicalReduction>
-        <hardwareInterface>${interface}</hardwareInterface>
       </actuator>
     </transmission>

Commit message: Addition of Transmission element

File: etarobtest/urdf/base.urdf.xacro (robot description, xacro)
@@ -134,34 +134,65 @@
   </xacro:macro>
   <!-- arm_connection_upper -->
-  <xacro:macro name="arm_connection_upper" params="suffix *origin rot_axis">
-    <joint name="${suffix}_upper_joint" type="revolute">
-      <axis xyz="0 ${rot_axis} 0" />
-      <limit lower="${-10*M_PI/180.0}" upper="${10*M_PI/180.0}" effort="${10*mx160_effort}" velocity="${mx160_velocity/5}"/>
-      <parent link="${suffix}_connection_upper"/>
-      <child link="${suffix}_arm" />
-      <xacro:insert_block name="origin" />
-    </joint>
-    <xacro:simple_transmission name="${suffix}_upper_joint" interface="hardware_interface/EffortJointInterface" />
-    <link name="${suffix}_arm">
-      <inertial>
-        <mass value="2.0" />
-        <origin xyz="0 0 0" />
-        <box_inertia m="2.0" x="${arm_width}" y="${arm_length}" z="${arm_height}" />
-      </inertial>
-      <visual>
-        <origin xyz="0 0 0" rpy="0 0 0" />
-        <geometry>
-          <mesh filename="package://etarobtest/meshes/arm_${suffix}_shifted.stl" />
-        </geometry>
-      </visual>
-      <collision>
-        <origin xyz="0 0 0" rpy="0 0 0" />
-        <geometry>
-          <box size="${arm_width} ${arm_length} ${arm_height}" />
-        </geometry>
-      </collision>
-    </link>
-  </xacro:macro>
-  <!--arm_connection_lower-->
+  <xacro:macro name="arm_connection_upper" params="suffix *origin rot_axis mimic">
+    <xacro:if value="${(mimic == 'false')}">
+      <joint name="${suffix}_upper_joint" type="revolute">
+        <axis xyz="0 ${rot_axis} 0" />
+        <limit lower="${-10*M_PI/180.0}" upper="${10*M_PI/180.0}" effort="${10*mx160_effort}" velocity="${mx160_velocity/5}"/>
+        <parent link="${suffix}_connection_upper"/>
+        <child link="${suffix}_arm" />
+        <xacro:insert_block name="origin" />
+      </joint>
+      <xacro:simple_transmission name="${suffix}_upper_joint" interface="hardware_interface/EffortJointInterface" />
+      <link name="${suffix}_arm">
+        <inertial>
+          <mass value="2.0" />
+          <origin xyz="0 0 0" />
+          <box_inertia m="2.0" x="${arm_width}" y="${arm_length}" z="${arm_height}" />
+        </inertial>
+        <visual>
+          <origin xyz="0 0 0" rpy="0 0 0" />
+          <geometry>
+            <mesh filename="package://etarobtest/meshes/arm_${suffix}_shifted.stl" />
+          </geometry>
+        </visual>
+        <collision>
+          <origin xyz="0 0 0" rpy="0 0 0" />
+          <geometry>
+            <box size="${arm_width} ${arm_length} ${arm_height}" />
+          </geometry>
+        </collision>
+      </link>
+    </xacro:if>
+    <xacro:if value="${(mimic == 'true')}">
+      <joint name= "${suffix}_lower_joint" type="revolute">
+        <axis xyz="0 ${rot_axis} 0" />
+        <limit lower="${-10*M_PI/180.0}" upper="${10*M_PI/180.0}" effort="${10*mx160_effort}" velocity="${mx160_velocity/5}"/>
+        <parent link="${suffix}_connection_lower"/>
+        <child link="${suffix}_arm" />
+        <xacro:insert_block name="origin" />
+      </joint>
+      <xacro:simple_transmission name="${suffix}_lower_joint" interface="hardware_interface/EffortJointInterface" />
+      <link name="${suffix}_arm">
+        <inertial>
+          <mass value="2.0" />
+          <origin xyz="0 0 0" />
+          <box_inertia m="2.0" x="${arm_width}" y="${arm_length}" z="${arm_height}" />
+        </inertial>
+        <visual>
+          <origin xyz="0 0 0" rpy="0 0 0" />
+          <geometry>
+            <mesh filename="package://etarobtest/meshes/arm_${suffix}_shifted.stl" />
+          </geometry>
+        </visual>
+        <collision>
+          <origin xyz="0 0 0" rpy="0 0 0" />
+          <geometry>
+            <box size="${arm_width} ${arm_length} ${arm_height}" />
+          </geometry>
+        </collision>
+      </link>
+    </xacro:if>
+  </xacro:macro>
+  <!--arm_connection_lower
   <xacro:macro name= "arm_connection_lower" params="suffix *origin rot_axis">
     <joint name= "${suffix}_lower_joint" type="revolute">
@@ -173,5 +204,5 @@
     </joint>
     <xacro:simple_transmission name="${suffix}_lower_joint" interface="hardware_interface/EffortJointInterface" />
-  </xacro:macro>
+  </xacro:macro> -->
   <!-- wheel -->
   <xacro:macro name="odom_wheel_tire" params="*origin suffix rot_axis_wheel">
@@ -229,14 +260,26 @@
     <origin xyz="0 0 0" rpy="0 0 0" />
   </xacro:base_lower>
-  <xacro:arm_connection_upper suffix="fl" rot_axis="1" >
+  <xacro:arm_connection_upper suffix="fl" rot_axis="1"  mimic="false">
     <origin xyz="-1.355178 0.214831 1.085205" rpy="0 0 0" />
   </xacro:arm_connection_upper>
-  <xacro:arm_connection_upper suffix="fr" rot_axis="-1" >
+  <xacro:arm_connection_upper suffix="fr" rot_axis="-1" mimic="false">
     <origin xyz="-1.35248 0.173899 -1.01988" rpy="0 0 0" />
   </xacro:arm_connection_upper>
-  <xacro:arm_connection_upper suffix="bl" rot_axis="1" >
+  <xacro:arm_connection_upper suffix="bl" rot_axis="1" mimic="false">
     <origin xyz="1.186923 0.173899 1.083927" rpy="0 0 0" />
   </xacro:arm_connection_upper>
-  <xacro:arm_connection_upper suffix="br" rot_axis="1" >
+  <xacro:arm_connection_upper suffix="br" rot_axis="1" mimic="false">
+    <origin xyz="1.194088 0.214831 -1.006421" rpy="0 0 0" />
+  </xacro:arm_connection_upper>
+  <xacro:arm_connection_upper suffix="fl" rot_axis="1"  mimic="true">
+    <origin xyz="-1.355178 0.214831 1.085205" rpy="0 0 0" />
+  </xacro:arm_connection_upper>
+  <xacro:arm_connection_upper suffix="fr" rot_axis="-1" mimic="true">
+    <origin xyz="-1.35248 0.173899 -1.01988" rpy="0 0 0" />
+  </xacro:arm_connection_upper>
+  <xacro:arm_connection_upper suffix="bl" rot_axis="1" mimic="true">
+    <origin xyz="1.186923 0.173899 1.083927" rpy="0 0 0" />
+  </xacro:arm_connection_upper>
+  <xacro:arm_connection_upper suffix="br" rot_axis="1" mimic="true">
     <origin xyz="1.194088 0.214831 -1.006421" rpy="0 0 0" />
   </xacro:arm_connection_upper>
@@ -244,5 +287,5 @@
   <xacro:arm_connection_lower suffix="fr" rot_axis="-1" />
   <xacro:arm_connection_lower suffix="bl" rot_axis="1" />
-  <xacro:arm_connection_lower suffix="br" rot_axis="1" />-->
+  <xacro:arm_connection_lower suffix="br" rot_axis="1" />
   <xacro:arm_connection_lower suffix="fl" rot_axis="1" >
     <origin xyz="0 0 0" rpy="0 0 0" />
@@ -256,5 +299,5 @@
   <xacro:arm_connection_lower suffix="br" rot_axis="1" >
     <origin xyz="0 0 0" rpy="0 0 0" />
-  </xacro:arm_connection_lower>
+  </xacro:arm_connection_lower>-->
   <!--<xacro:arm_connection_upper suffix="fl" rot_axis="1" >
     <origin xyz="0 0 0" rpy="0 0 0" />

Commit message: Addition of Transmission elements

File: etarobtest/urdf/base.urdf.xacro (robot description, xacro)
@@ -95,4 +95,10 @@
 	</geometry>
       </visual>
+      <visual>
+        <origin xyz="0 0 0" rpy="0 0 0" />
+	<geometry>
+	  <mesh filename="package://etarobtest/meshes/lower_connection_${suffix}.stl" />
+	</geometry>
+      </visual>
       <collision>
         <origin xyz="0 0 0" rpy="0 0 0" />
@@ -103,5 +109,5 @@
     </link>
   </xacro:macro>
-  <!-- base_connection (lower) -->
+  <!-- base_connection (lower)
   <xacro:macro name= "base_lower" params="suffix *origin rot_axis">
     <joint name= "${suffix}_base_lower" type="revolute">
@@ -132,6 +138,6 @@
       </collision>
     </link>
-  </xacro:macro>
-  <!-- arm_connection_upper -->
+  </xacro:macro>-->
+  <!-- arm_connection_upper-->
   <xacro:macro name="arm_connection_upper" params="suffix *origin rot_axis mimic">
     <xacro:if value="${(mimic == 'false')}">
@@ -140,9 +146,9 @@
         <limit lower="${-10*M_PI/180.0}" upper="${10*M_PI/180.0}" effort="${10*mx160_effort}" velocity="${mx160_velocity/5}"/>
         <parent link="${suffix}_connection_upper"/>
-        <child link="${suffix}_arm" />
+        <child link="${suffix}_arm_upper" />
         <xacro:insert_block name="origin" />
       </joint>
       <xacro:simple_transmission name="${suffix}_upper_joint" interface="hardware_interface/EffortJointInterface" />
-      <link name="${suffix}_arm">
+      <link name="${suffix}_arm_upper">
         <inertial>
           <mass value="2.0" />
@@ -164,14 +170,14 @@
       </link>
     </xacro:if>
-    <xacro:if value="${(mimic == 'true')}">
+    <!--<xacro:if value="${(mimic == 'true')}">
       <joint name= "${suffix}_lower_joint" type="revolute">
         <axis xyz="0 ${rot_axis} 0" />
         <limit lower="${-10*M_PI/180.0}" upper="${10*M_PI/180.0}" effort="${10*mx160_effort}" velocity="${mx160_velocity/5}"/>
         <parent link="${suffix}_connection_lower"/>
-        <child link="${suffix}_arm" />
+        <child link="${suffix}_arm_upper" />
         <xacro:insert_block name="origin" />
       </joint>
-      <xacro:simple_transmission name="${suffix}_lower_joint" interface="hardware_interface/EffortJointInterface" />
-      <link name="${suffix}_arm">
+      <xacro:simple_transmission name="${suffix}_lower_joint" interface="hardware_interface/EffortJointInterface" />-->
+      <!--<link name="${suffix}_arm_lower">
         <inertial>
           <mass value="2.0" />
@@ -192,5 +198,5 @@
         </collision>
       </link>
-    </xacro:if>
+    </xacro:if>-->
   </xacro:macro>
   <!--arm_connection_lower
@@ -212,5 +218,5 @@
       <dynamics damping="0.0" friction="0.0" />
       <xacro:insert_block name="origin"/>
-      <parent link="${suffix}_arm" />
+      <parent link="${suffix}_arm_upper" />
       <child link="${suffix}_wheel_link" />
     </joint>
@@ -239,5 +245,5 @@
     <origin xyz="0 0 0" rpy="0 0 0" />
   </xacro:base_upper>
-  <xacro:base_upper suffix="fr" rot_axis="-1" >
+  <xacro:base_upper suffix="fr" rot_axis="1" >
     <origin xyz="0 0 0" rpy="0 0 0" />
   </xacro:base_upper>
@@ -248,5 +254,5 @@
     <origin xyz="0 0 0" rpy="0 0 0" />
   </xacro:base_upper>
-  <xacro:base_lower suffix="fl" rot_axis="2" >
+  <!--<xacro:base_lower suffix="fl" rot_axis="2" >
     <origin xyz="0 0 0" rpy="0 0 0" />
   </xacro:base_lower>
@@ -259,5 +265,5 @@
   <xacro:base_lower suffix="br" rot_axis="1" >
     <origin xyz="0 0 0" rpy="0 0 0" />
-  </xacro:base_lower>
+  </xacro:base_lower>-->
   <xacro:arm_connection_upper suffix="fl" rot_axis="1"  mimic="false">
     <origin xyz="-1.355178 0.214831 1.085205" rpy="0 0 0" />
@@ -272,8 +278,8 @@
     <origin xyz="1.194088 0.214831 -1.006421" rpy="0 0 0" />
   </xacro:arm_connection_upper>
-  <xacro:arm_connection_upper suffix="fl" rot_axis="1"  mimic="true">
+  <!--<xacro:arm_connection_upper suffix="fl" rot_axis="1"  mimic="true">
     <origin xyz="-1.355178 0.214831 1.085205" rpy="0 0 0" />
-  </xacro:arm_connection_upper>
-  <xacro:arm_connection_upper suffix="fr" rot_axis="-1" mimic="true">
+  </xacro:arm_connection_upper>-->
+  <!--<xacro:arm_connection_upper suffix="fr" rot_axis="-1" mimic="true">
     <origin xyz="-1.35248 0.173899 -1.01988" rpy="0 0 0" />
   </xacro:arm_connection_upper>
@@ -283,5 +289,5 @@
   <xacro:arm_connection_upper suffix="br" rot_axis="1" mimic="true">
     <origin xyz="1.194088 0.214831 -1.006421" rpy="0 0 0" />
-  </xacro:arm_connection_upper>
+  </xacro:arm_connection_upper>-->
     <!--<xacro:arm_connection_lower suffix="fl" rot_axis="1" />
   <xacro:arm_connection_lower suffix="fr" rot_axis="-1" />

Commit message: Integration of sensors

File: etarobtest/urdf/base.urdf.xacro (robot description, xacro)
@@ -45,4 +45,24 @@
                 iyy="${m*(z*z+x*x)/12}" iyz = "0" izz="${m*(x*x+y*y)/12}" />
   </xacro:macro>
+  <!-- gps sensor -->
+  <xacro:property name="reach_mass" value="0.69" />
+  <xacro:property name="reach_radius" value="0.095" />
+  <xacro:property name="reach_height" value="0.19" />
+  <xacro:property name="reach_origin_x" value="0.562" />
+  <xacro:property name="reach_origin_y" value="0.0" />
+  <xacro:property name="reach_origin_z" value="1.454" />
+  <xacro:property name="reach_collision_origin_x" value="0.0" />
+  <xacro:property name="reach_collision_origin_y" value="0.0" />
+  <xacro:property name="reach_collision_origin_z" value="-0.0125" />
+  <xacro:property name="gps_mass" value="0.69" />
+  <xacro:property name="gps_length" value="0.095" />
+  <xacro:property name="gps_width" value="0.095" />
+  <xacro:property name="gps_height" value="0.19" />
+  <xacro:property name="gps_origin_x" value="0.562" />
+  <xacro:property name="gps_origin_y" value="0.0" />
+  <xacro:property name="gps_origin_z" value="1.454" />
+  <xacro:property name="gps_collision_origin_x" value="0.0" />
+  <xacro:property name="gps_collision_origin_y" value="0.0" />
+  <xacro:property name="gps_collision_origin_z" value="-0.0125" />
   <!-- base_footprint -->
   <link name="base_footprint" />
@@ -242,4 +262,51 @@
     <xacro:gazebo_wheel_link name="${suffix}_wheel_link"/>
   </xacro:macro>
+  <!-- gps sensor -->
+  <xacro:macro name="gps" params="*origin parent_link gps_name update_rate refLat refLon refHead refAlt show_visual" >
+    <joint name="base_to_gps" type="fixed">
+      <xacro:insert_block name="origin" />
+      <parent link="${parent_link}" />
+      <child link="${gps_name}_link"/>
+    </joint>
+    <link name="${gps_name}_link">
+      <inertial>
+        <origin xyz="0 0 0" rpy="0 0 0" />
+        <mass value="${reach_mass}" />
+        <xacro:cylinder_inertia m="${reach_mass}" r="${reach_radius}" h="${reach_height}" />
+      </inertial>
+      <xacro:if value="${show_visual}" >
+        <visual>
+          <geometry>
+            <mesh filename="package://etarobtest/meshes/sensors/sensor.stl" />
+          </geometry>
+        </visual>
+      </xacro:if>
+      <collision>
+        <origin xyz="${reach_collision_origin_x} ${gps_collision_origin_y} ${gps_collision_origin_z}"
+                rpy="0 0 0" />
+        <geometry>
+          <cylinder radius="${reach_radius}" length="${reach_height}" />
+        </geometry>
+      </collision>
+    </link>
+    <gazebo>
+      <plugin name="${gps_name}_plugin" filename="libhector_gazebo_ros_gps.so">
+        <updateRate>${update_rate}</updateRate>
+        <bodyName>${gps_name}_link</bodyName>
+        <robotNamespace>etarob</robotNamespace>
+        <frameId>base_link</frameId>
+        <topicName>/${gps_name}_link/fix</topicName>
+        <velocityTopicName>/${gps_name}_link/fix_velocity</velocityTopicName>
+        <referenceLatitude>${refLat}</referenceLatitude>
+        <referenceLongitude>${refLon}</referenceLongitude>
+        <referenceAltitude>${refAlt}</referenceAltitude>
+        <referenceHeading>${refHead}</referenceHeading>
+        <drift>0.0 0.0 0.0</drift>
+        <gaussianNoise>0.00 0.00 0.00</gaussianNoise>
+        <velocityDrift>0 0 0</velocityDrift>
+        <velocityGaussianNoise>0.00 0.00 0.00</velocityGaussianNoise>
+      </plugin>
+    </gazebo>
+  </xacro:macro>
   <xacro:base_upper suffix="fl" rot_axis="1" >
     <origin xyz="0 0 0" rpy="0 0 0" />
@@ -342,3 +409,6 @@
     <origin xyz="0 0 0" rpy="0 0 0" />
   </xacro:odom_wheel_tire>-->
+  <xacro:gps parent_link="base_link" gps_name="gps_rover" update_rate="50" refLat="50.761127" refLon="6.074315" refAlt="0.0" refHead="90" show_visual="true" >
+    <origin xyz="0 0 0" rpy="0.0 0.0 0.0" />
+  </xacro:gps>
 </robot>

File: etarobtest/urdf/test.gazebo.xacro (robot description, xacro)
@@ -19,4 +19,17 @@
       <xyzOffset>0.0 0.0 0.0</xyzOffset>
       <updateRate>50.0</updateRate>
+    </plugin>
+  </gazebo>
+  <!-- p3d_base_controller -->
+  <gazebo>
+    <plugin name="p3d_base_controller" filename="libgazebo_ros_p3d.so">
+      <alwaysOn>true</alwaysOn>
+      <updateRate>50.0</updateRate>
+      <bodyName>base_link</bodyName>
+      <topicName>ground_truth/state</topicName>
+      <gaussianNoise>0.01</gaussianNoise>
+      <frameName>world</frameName>
+      <xyzOffsets>0 0 0</xyzOffsets>
+      <rpyOffsets>0 0 0</rpyOffsets>
     </plugin>
   </gazebo>
